File: kiCAD/PCB IREC 2025.kicad_pcb (KiCad board)
At the start: 2 copper layers, 0 parts

Commit message: Add files via upload
Parts:
- added 5V1: Power_Hole, TestPoint:TestPoint_THTPad_2.5x2.5mm_Drill1.2mm, F.Cu at (175.4, 52.1)
- added ADXL375: ADXL375, SACCUP-2025:ADXL375, F.Cu at (145.8, 74.5)
- added BMP280: ~, SACCUP-2025:BMP280, F.Cu at (148.1, 55.2)
- added Component_Breakout1: ~, SACCUP-2025:Component Breakout, F.Cu at (173.2, 51.9)
- added DS1307: ~, SACCUP-2025:DS1307, F.Cu at (146.0, 128.6)
- added G***: LOGO, SACCUP-2025:SLURPL-Logo, F.Cu at (192.5, 69.5)
- added GND1: Power_Hole, TestPoint:TestPoint_THTPad_2.5x2.5mm_Drill1.2mm, F.Cu at (179.4, 52.1)
- added INA219: ~, SACCUP-2025:INA219, F.Cu at (168.4, 55.4)
- added LSM9DS1: ~, SACCUP-2025:LSM9DS1, F.Cu at (175.0, 135.1)
- added MPU6050: ~, SACCUP-2025:MPU6050, F.Cu at (147.1, 63.0)
- added RX1: 10K, Resistor_THT:R_Axial_DIN0207_L6.3mm_D2.5mm_P10.16mm_Horizontal, F.Cu at (176.1, 83.5)
- added RX2: 10K, Resistor_THT:R_Axial_DIN0207_L6.3mm_D2.5mm_P10.16mm_Horizontal, F.Cu at (166.0, 87.0)
- added SCL0: 4.7K, Resistor_THT:R_Axial_DIN0207_L6.3mm_D2.5mm_P10.16mm_Horizontal, F.Cu at (165.9, 90.5)
- added SCL1: 4.7K, Resistor_THT:R_Axial_DIN0207_L6.3mm_D2.5mm_P10.16mm_Horizontal, F.Cu at (165.9, 94.0)
- added SCL2: 4.7K, Resistor_THT:R_Axial_DIN0207_L6.3mm_D2.5mm_P10.16mm_Horizontal, F.Cu at (165.9, 97.5)
- added SDA0: 4.7K, Resistor_THT:R_Axial_DIN0207_L6.3mm_D2.5mm_P10.16mm_Horizontal, F.Cu at (182.3, 83.5)
- added SDA1: 4.7K, Resistor_THT:R_Axial_DIN0207_L6.3mm_D2.5mm_P10.16mm_Horizontal, F.Cu at (182.3, 87.5)
- added SDA2: 4.7K, Resistor_THT:R_Axial_DIN0207_L6.3mm_D2.5mm_P10.16mm_Horizontal, F.Cu at (182.3, 91.6)
- added TX1: 10K, Resistor_THT:R_Axial_DIN0207_L6.3mm_D2.5mm_P10.16mm_Horizontal, F.Cu at (182.3, 95.7)
- added TX2: 10K, Resistor_THT:R_Axial_DIN0207_L6.3mm_D2.5mm_P10.16mm_Horizontal, F.Cu at (182.3, 99.7)
- added U1: Teensy4.1, SACCUP-2025:Teensy41, F.Cu at (135.4, 95.6)
Routing:
- net /3V3: track 0.00 -> 223.4 mm, vias 0 -> 4
- net GND: track 0.00 -> 170.1 mm, vias 0 -> 3
- net /SDA0: track 0.00 -> 150.8 mm, vias 0 -> 3
- net /SCL0: track 0.00 -> 137.4 mm, vias 0 -> 4
- net /SDA2: track 0.00 -> 126.2 mm, vias 0 -> 3
- net /TX2: track 0.00 -> 120.2 mm, vias 0 -> 3
- net /SCL1: track 0.00 -> 118.7 mm, vias 0 -> 3
- net /TX1: track 0.00 -> 113.6 mm, vias 0 -> 5
- net /SDA1: track 0.00 -> 110.0 mm, vias 0 -> 2
- net /SCL2: track 0.00 -> 102.8 mm, vias 0 -> 2
- net /RFM-RST: track 0.00 -> 87.9 mm, vias 0 -> 2
- net /RX1: track 0.00 -> 85.1 mm, vias 0 -> 3
- net /RFM-MISO: track 0.00 -> 81.4 mm, vias 0 -> 1
- net /RX2: track 0.00 -> 78.8 mm, vias 0 -> 2
- net /RFM-CS: track 0.00 -> 65.3 mm, vias 0 -> 2
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- added copper zone on B.Cu, net (none)
- added copper zone on F.Cu, net (none)
Other:
- board outline added: 72.5 x 87.5 mm
- board text added: "THE MISSLE KNOWS WHERE IT IS.."

Commit message: Add files via upload
Parts:
- moved U1 2.16 mm to (135.4, 97.8)
- moved MPU6050 1.52 mm to (147.1, 64.5)
- moved DS1307 1.34 mm to (146.0, 130.0)
Routing:
- net /SDA0: track 150.8 -> 146.9 mm
- net /RFM-MOSI: track 63.7 -> 67.3 mm
- net /SCL0: track 137.4 -> 140.6 mm
- net GND: track 170.1 -> 173.2 mm, vias 3 -> 5
- net /SDA2: track 126.2 -> 128.9 mm
- net +5V: track 47.0 -> 49.6 mm
- net /TX2: track 120.2 -> 122.5 mm
- net /RFM-CS: track 65.3 -> 67.3 mm
- net /SCL2: track 102.8 -> 104.8 mm
- net /RFM-RST: track 87.9 -> 89.8 mm
- net /RFM-INT: track 62.8 -> 64.5 mm
- net /TX1: track 113.6 -> 112.1 mm, vias 5 -> 6
- net /SCL1: track 118.7 -> 120.0 mm
- net /RFM-MISO: track 81.4 -> 82.6 mm
- net /3V3: track 223.4 -> 224.1 mm
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